File: Radio/Radio.kicad_sch (KiCad schematic)
At the start: 2 parts, among them IC1 SI4844-A10-GU

Commit message: Update Radio.kicad_sch
Did basic Schematic
Parts:
- added AE1: Antenna, symbol Device:Antenna
- added C10, C11, C12, C14, C15, C3, C4, C5, C6, C7, C8, C9: C, symbol Device:C
- added FB1: 2.5K, symbol Device:FerriteBead
- added L1: AM_ANT, symbol Device:L_Ferrite
- added L2: 270nH, symbol Device:L
- added Q1: NPN, symbol Simulation_SPICE:NPN
- added R1, R2, R3, R4, R5, R6, R7, R8: R, symbol Device:R
- added RV1: 100K, symbol Device:R_Potentiometer
- added Y1: 32.768 kHz, symbol Device:Crystal
Connections:
- net RST: now reaches A1.13 (D10)
- net RST: now also IC1.15 (~{RST}), C7.2, R4.2
- net +3V3: now reaches A1.17 (3V3)
- net +3V3: now also IC1.20 (VDD1), IC1.21 (VDD2), IC1.5 (BAND), C11.1, C5.1, C6.1, R1.1, R2.1, R4.1, R5.1
- net SDIO: now reaches A1.23 (SDA/A4)
- net SDIO: now also IC1.16 (SDIO), R2.2
- net SCLK: now reaches A1.24 (SCL/A5)
- net SCLK: now also IC1.17 (SCLK), R1.2
- net GND: now reaches A1.29 (GND), A1.4 (GND)
- net GND: now also IC1.10 (NC_3), IC1.11 (NC_4), IC1.13 (GND_1), IC1.14 (GND_2), IC1.9 (RFGND), C11.2, C12.2, C3.1, C4.1, C7.1, C8.2, C9.2, L1.1, L2.2, Q1.3 (E), R7.2, R8.1
- net IRQ: now reaches A1.5 (D2)
- net IRQ: now also IC1.2 (IRQ)
- net LNA: now reaches IC1.1 (LNA_EN)
- net LNA: now also R6.1
- net at IC1.12 (AMI): now also C10.1
- net XTAL1: now reaches IC1.18 (XTALO)
- net XTAL1: now also C3.2, Y1.2
- net XTAL2: now reaches IC1.19 (XTALI)
- net XTAL2: now also C4.2, Y1.1
- net at IC1.22 (DBYP): now also C5.2, C6.2
- net TUNE1: now reaches IC1.3 (TUNE1)
- net TUNE1: now also C8.1, C9.1, RV1.1
- net TUNE2: now reaches IC1.4 (TUNE2)
- net TUNE2: now also RV1.2
- net FM_ANT: now reaches IC1.8 (FMI)
- net FM_ANT: now also C15.1, L2.1
- new net: C14.1, Q1.2 (B), R6.2, R7.1
- new net: R8.2, RV1.3
- new net: C12.1, R3.1, R5.2
- new net: C15.2, Q1.1 (C), R3.2
- new net: C14.2, FB1.2
- new net AM_ANT: AE1.1 (A), C10.2, FB1.1, L1.2
Other:
- note added: "Antenna"
- note added: "Arduino Nano"
- note added: "Crystal"
- note added: "SI4844-A10-GU"
- note added: "Tuning Resistor aka potentiometer"
- moved on the sheet: A1, IC1

Commit message: prepped the base PCB
This is my 1st RF pcb so I just did the placement for now

I am gonna consult an engineer later to see what I have wrong
Parts:
- removed A1: Arduino_Nano_Every, Module:Arduino_Nano, symbol MCU_Module:Arduino_Nano_Every
- removed L1: AM_ANT, symbol Device:L_Ferrite
- added C1, C2: 4.7uF, Capacitor_SMD:C_0603_1608Metric_Pad1.08x0.95mm_HandSolder, symbol Device:C
- added J1: AudioJack3, Connector_Audio:Jack_3.5mm_CUI_SJ1-3523N_Horizontal, symbol Connector_Audio:AudioJack3
- added J2: Conn_01x04_Pin, DM-OLED096-636:MODULE_DM-OLED096-636, symbol Connector:Conn_01x04_Pin
- added J3: Conn_01x02_Pin, Connector:FanPinHeader_1x03_P2.54mm_Vertical, symbol Connector:Conn_01x02_Pin
- added U1: ARDUINO_PRO_MINI, ARDUINO_PRO_MINI:MODULE_ARDUINO_PRO_MINI, symbol ARDUINO_PRO_MINI:ARDUINO_PRO_MINI
- AE1: footprint (none) -> Connector_Coaxial:SMA_Amphenol_901-143_Horizontal; symbol Device:Antenna -> Device:Antenna_Shield
- C10, C11: value C -> 0.47uF; footprint (none) -> Capacitor_SMD:C_0603_1608Metric_Pad1.08x0.95mm_HandSolder
- C12, C14: value C -> 33nF; footprint (none) -> Capacitor_SMD:C_0603_1608Metric_Pad1.08x0.95mm_HandSolder
- C15: value C -> 10pF; footprint (none) -> Capacitor_SMD:C_0603_1608Metric_Pad1.08x0.95mm_HandSolder
- C3, C4: value C -> 22pF; footprint (none) -> Capacitor_SMD:C_0603_1608Metric_Pad1.08x0.95mm_HandSolder
- C5: value C -> 4.7uF; footprint (none) -> Capacitor_SMD:C_0603_1608Metric_Pad1.08x0.95mm_HandSolder
- C6, C7, C9: value C -> 0.1uF; footprint (none) -> Capacitor_SMD:C_0603_1608Metric_Pad1.08x0.95mm_HandSolder
- C8: value C -> 47uF; footprint (none) -> Capacitor_SMD:C_0603_1608Metric_Pad1.08x0.95mm_HandSolder
- FB1: footprint (none) -> Resistor_SMD:R_0805_2012Metric_Pad1.20x1.40mm_HandSolder
- IC1: footprint SOP64P600X175-24N -> RadioLib:SOP64P600X175-24N
- L2: footprint (none) -> Inductor_SMD:L_0603_1608Metric_Pad1.05x0.95mm_HandSolder
- Q1: footprint (none) -> RadioLib:SS9018
- R1, R2: value R -> 2.2K; footprint (none) -> Resistor_SMD:R_0603_1608Metric_Pad0.98x0.95mm_HandSolder
- R3: value R -> 1K; footprint (none) -> Resistor_SMD:R_0603_1608Metric_Pad0.98x0.95mm_HandSolder
- R4, R7: value R -> 100K; footprint (none) -> Resistor_SMD:R_0603_1608Metric_Pad0.98x0.95mm_HandSolder
- R5: value R -> 10; footprint (none) -> Resistor_SMD:R_0603_1608Metric_Pad0.98x0.95mm_HandSolder
- R6: value R -> 120K; footprint (none) -> Resistor_SMD:R_0603_1608Metric_Pad0.98x0.95mm_HandSolder
- R8: value R -> 100; footprint (none) -> Resistor_SMD:R_0603_1608Metric_Pad0.98x0.95mm_HandSolder
- RV1: footprint (none) -> Potentiometer_THT:Potentiometer_Alpha_RD901F-40-00D_Single_Vertical
- Y1: footprint (none) -> Crystal:Crystal_HC49-4H_Vertical
Connections:
- net +3V3: now also J2.1 (Pin_1), U1.JP1_4 (VCC), U1.JP6_4 (VCC_1)
- net AM_ANT: now also J3.1 (Pin_1)
- net GND: now also AE1.2 (Shield), J1.S, J2.2 (Pin_2), J3.2 (Pin_2), U1.JP1_5 (GND), U1.JP1_6 (GND), U1.JP6_2 (GND_1), U1.JP7_9 (GND_2)
- net IRQ: now also U1.JP7_8 (D2)
- net RST: now also U1.JP6_10 (MISO)
- net SCLK: now also J2.4 (Pin_4), U1.JP2_2 (A5)
- net SDIO: now also J2.3 (Pin_3), U1.JP2_1 (A4)
- net at IC1.23 (ROUT): now also C2.1
- net at IC1.24 (LOUT): now also C1.1
- new net: C1.2, J1.T
- new net: C2.2, J1.R

Commit message: Update PCB: move components
Moved several components to new positions. and changed potentiometer footprint
Parts:
- removed J3: Conn_01x02_Pin, Connector:FanPinHeader_1x03_P2.54mm_Vertical, symbol Connector:Conn_01x02_Pin
- added J3: Conn_01x02_Socket, Connector_PinHeader_2.54mm:PinHeader_1x02_P2.54mm_Vertical, symbol Connector:Conn_01x02_Socket
- added J4: Conn_01x07_Pin, Connector_PinHeader_2.54mm:PinHeader_1x07_P2.54mm_Vertical, symbol Connector:Conn_01x07_Pin
- added L1: L_Ferrite_Small, Connector_PinHeader_2.54mm:PinHeader_1x02_P2.54mm_Horizontal, symbol Device:L_Ferrite_Small
- RV1: footprint Potentiometer_THT:Potentiometer_Alpha_RD901F-40-00D_Single_Vertical -> RadioLib:RK09L1120A2S
Connections:
- net +3V3: now also J3.2 (Pin_2)
- net AM_ANT: now also L1.2
- net GND: now also J3.1 (Pin_1), L1.1
- net TUNE1: now also RV1.3; no longer RV1.1
- net at R8.2: now also RV1.1; no longer RV1.3
- net ROW1: now reaches U1.JP7_1 (D9)
- net ROW1: now also J4.7 (Pin_7)
- net ROW2: now reaches U1.JP7_2 (D8)
- net ROW2: now also J4.6 (Pin_6)
- net ROW3: now reaches U1.JP7_3 (D7)
- net ROW3: now also J4.5 (Pin_5)
- net ROW4: now reaches U1.JP7_4 (D6)
- net ROW4: now also J4.4 (Pin_4)
- net COL1: now reaches U1.JP7_5 (D5)
- net COL1: now also J4.3 (Pin_3)
- net COL2: now reaches U1.JP7_6 (D4)
- net COL2: now also J4.2 (Pin_2)
- net COL3: now reaches U1.JP7_7 (D3)
- net COL3: now also J4.1 (Pin_1)
Other:
- note added: "I/O and Power"
- moved on the sheet: J2, RV1

Commit message: Update PCB layout and footprints
Parts:
- J2: footprint DM-OLED096-636:MODULE_DM-OLED096-636 -> Connector_PinHeader_2.54mm:PinHeader_1x04_P2.54mm_Vertical
- RV1: footprint RadioLib:RK09L1120A2S -> Potentiometer_THT:Potentiometer_Alps_RK163_Single_Horizontal
Changed lines of the file:
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@@
 			)
 		)
-		(property "Footprint" "DM-OLED096-636:MODULE_DM-OLED096-636"
+		(property "Footprint" "Connector_PinHeader_2.54mm:PinHeader_1x04_P2.54mm_Vertical"
 			(at 356.87 151.13 0)
 			(effects
@@
 			)
 		)
-		(property "Footprint" "RadioLib:RK09L1120A2S"
+		(property "Footprint" "Potentiometer_THT:Potentiometer_Alps_RK163_Single_Horizontal"
 			(at 41.91 46.99 0)
 			(effects

Commit message: Updated PCB
Parts:
- removed C5: 4.7uF, Capacitor_SMD:C_0603_1608Metric_Pad1.08x0.95mm_HandSolder, symbol Device:C
- removed C6, C7, C9: 0.1uF, Capacitor_SMD:C_0603_1608Metric_Pad1.08x0.95mm_HandSolder, symbol Device:C
- removed C8: 47uF, Capacitor_SMD:C_0603_1608Metric_Pad1.08x0.95mm_HandSolder, symbol Device:C
- removed IC1: SI4844-A10-GU, RadioLib:SOP64P600X175-24N, symbol SamacSys_Parts:SI4844-A10-GU
- removed J3: Conn_01x02_Socket, Connector_PinHeader_2.54mm:PinHeader_1x02_P2.54mm_Vertical, symbol Connector:Conn_01x02_Socket
- removed J4: Conn_01x07_Pin, Connector_PinHeader_2.54mm:PinHeader_1x07_P2.54mm_Vertical, symbol Connector:Conn_01x07_Pin
- removed R1, R2: 2.2K, Resistor_SMD:R_0603_1608Metric_Pad0.98x0.95mm_HandSolder, symbol Device:R
- removed R4: 100K, Resistor_SMD:R_0603_1608Metric_Pad0.98x0.95mm_HandSolder, symbol Device:R
- removed R6: 120K, Resistor_SMD:R_0603_1608Metric_Pad0.98x0.95mm_HandSolder, symbol Device:R
- removed R8: 100, Resistor_SMD:R_0603_1608Metric_Pad0.98x0.95mm_HandSolder, symbol Device:R
- removed RV1: 100K, Potentiometer_THT:Potentiometer_Alps_RK163_Single_Horizontal, symbol Device:R_Potentiometer
- removed U1: ARDUINO_PRO_MINI, ARDUINO_PRO_MINI:MODULE_ARDUINO_PRO_MINI, symbol ARDUINO_PRO_MINI:ARDUINO_PRO_MINI
- added C19: 22nF, Capacitor_SMD:C_0603_1608Metric_Pad1.08x0.95mm_HandSolder, symbol Device:C
- added C20: 100nF, Capacitor_SMD:C_0603_1608Metric_Pad1.08x0.95mm_HandSolder, symbol Device:C
- added D1, D2, D3, D4: 1N4148, Diode_THT:D_DO-35_SOD27_P7.62mm_Horizontal, symbol Diode:1N4148
- added R11, R12: 1k, Resistor_SMD:R_0603_1608Metric_Pad0.98x0.95mm_HandSolder, symbol Device:R
- added SW1: RotaryEncoder_Switch, Rotary_Encoder:RotaryEncoder_Alps_EC11E-Switch_Vertical_H20mm_CircularMountingHoles, symbol Device:RotaryEncoder_Switch
- added SW2, SW3, SW4: SW_Push_45deg, FSM8JH:SW_FSM8JH, symbol Switch:SW_Push_45deg
- added U1: Si4735-D60-GU, Package_SO:SSOP-24_3.9x8.7mm_P0.635mm, symbol RF_AM_FM:Si4735-D60-GU
- added U2: RP2040-ZERO, RP2040-ZERO:MODULE_RP2040-ZERO, symbol RP2040-ZERO:RP2040-ZERO
- added U5: PAM8301, Package_TO_SOT_SMD:SOT-23-6_Handsoldering, symbol Amplifier_Audio:PAM8301
- C1: value 4.7uF -> 10uF
- C2: value 4.7uF -> 0.1uF
- J2: footprint Connector_PinHeader_2.54mm:PinHeader_1x04_P2.54mm_Vertical -> DM-OLED096-636:MODULE_DM-OLED096-636
Connections:
- net +3V3: now also C1.1, C2.2, C19.2, C20.1, U1.20 (VD), U1.21 (VA), U2.21 (3V3), U5.5 (VDD)
- net COL1: now also D1.1 (K), D3.1 (K), U2.7 (GP6)
- net COL2: now also D2.1 (K), D4.1 (K), U2.10 (GP9)
- net FM_ANT: now also U1.8 (FMI)
- net GND: now also C1.2, C2.1, C20.2, SW1.C, U1.13 (GND), U1.14 (GND), U1.9 (RFGND), U2.22 (GND), U5.2 (GND)
- net ROW1: now also SW2.1, SW4.1, U2.8 (GP7)
- net ROW2: now also SW1.S1, SW3.1, U2.9 (GP8)
- net RST: now also U1.15 (~{RST}), U2.13 (GP12)
- net SCLK: now also U1.17 (SCLK), U2.15 (GP14); no longer J2.4 (Pin_4)
- net XTAL1: now also U1.19 (RCLK)
- net XTAL2: now also U1.3 (GPO3/[DCLK])
- net at J1.T: now also U5.6 (OUT+); no longer C1.2
- net at J1.R: now also U5.1 (OUT-); no longer C2.2
- net AM_ANT_IC: now reaches C10.1
- net AM_ANT_IC: now also U1.12 (AMI)
- net SDIO renamed SDA_OLED
- net SDA_OLED: now also U2.18 (GP27)
- new net: D2.2 (A), SW4.2
- new net: D4.2 (A), SW1.S2
- new net: R11.1, U1.23 (ROUT/[DOUT])
- new net: D3.2 (A), SW3.2
- new net: C19.1, U1.22 (DBYP)
- new net: R12.1, U1.24 (LOUT/[DFS])
- new net: D1.2 (A), SW2.2
- new net Aud_Enable: U2.20 (GP29), U5.4 (~{SD})
- new net Audio_Amp: R11.2, R12.2, U5.3 (IN)
- new net Enable: U1.16 (~{SEN}), U2.14 (GP13)
- new net Encoder 1: SW1.A, U2.11 (GP10)
- new net Encoder 2: SW1.B, U2.12 (GP11)
- new net SCLK_OLED: J2.4 (Pin_4), U2.17 (GP26)
- new net SDA: U1.18 (SDIO), U2.16 (GP15)
- new net VBUS: U2.23 (5V)
- no-connect marks 0 -> 2
Other:
- note added: "Audio Amp PAM8301"
- note added: "Encoder EC11"
- note added: "I/O"
- note added: "RP2040-Zero"
- note added: "Si4735 D60"
- note removed: "Arduino Nano"
- note removed: "I/O and Power"
- note removed: "SI4844-A10-GU"
- note removed: "Tuning Resistor aka potentiometer"
- moved on the sheet: J2

Commit message: push to git
Parts:
- removed C12: 33nF, Capacitor_SMD:C_0603_1608Metric_Pad1.08x0.95mm_HandSolder, symbol Device:C
- removed C15: 10pF, Capacitor_SMD:C_0603_1608Metric_Pad1.08x0.95mm_HandSolder, symbol Device:C
- removed Q1: NPN, RadioLib:SS9018, symbol Simulation_SPICE:NPN
- removed R11, R12: 1k, Resistor_SMD:R_0603_1608Metric_Pad0.98x0.95mm_HandSolder, symbol Device:R
- removed R3: 1K, Resistor_SMD:R_0603_1608Metric_Pad0.98x0.95mm_HandSolder, symbol Device:R
- removed R5: 10, Resistor_SMD:R_0603_1608Metric_Pad0.98x0.95mm_HandSolder, symbol Device:R
- removed R7: 100K, Resistor_SMD:R_0603_1608Metric_Pad0.98x0.95mm_HandSolder, symbol Device:R
- removed U5: PAM8301, Package_TO_SOT_SMD:SOT-23-6_Handsoldering, symbol Amplifier_Audio:PAM8301
- added C5, C6: 1uF, Capacitor_SMD:C_0603_1608Metric_Pad1.08x0.95mm_HandSolder, symbol Device:C
- added C7: 0.1uF, Capacitor_SMD:C_0603_1608Metric_Pad1.08x0.95mm_HandSolder, symbol Device:C
- added C8, C9: 0.39uF, Capacitor_SMD:C_0603_1608Metric_Pad1.08x0.95mm_HandSolder, symbol Device:C
- added D5, D6: CM1213A-01SO, Package_TO_SOT_SMD:SOT-23, symbol Power_Protection:CM1213A-01SO
- added FB2: 1k, Resistor_SMD:R_0805_2012Metric_Pad1.20x1.40mm_HandSolder, symbol Device:FerriteBead
- added J3: AudioJack3, Connector_Audio:Jack_3.5mm_CUI_SJ1-3523N_Horizontal, symbol Connector_Audio:AudioJack3
- added L3: 4.7uH, Inductor_SMD:L_0603_1608Metric_Pad1.05x0.95mm_HandSolder, symbol Device:L
- added R1, R2: 100, Resistor_SMD:R_0603_1608Metric_Pad0.98x0.95mm_HandSolder, symbol Device:R_Small
- added R4, R6, R8, R9: 20k, Resistor_SMD:R_0603_1608Metric_Pad0.98x0.95mm_HandSolder, symbol Device:R_Small
- added U3: PAM8302AAY, Package_DFN_QFN:DFN-8-1EP_3x3mm_P0.65mm_EP1.55x2.4mm, symbol Amplifier_Audio:PAM8302AAY
- added U4: LM4910MM, LM4910MM:SOP65P490X110-8N, symbol LM4910MM:LM4910MM
- added U5: PE4259, PE4259:SOT65P215X110-6N, symbol PE4259:PE4259
- C11: value 0.47uF -> 33pF
- C14: value 33nF -> 18pF
- L1: footprint Connector_PinHeader_2.54mm:PinHeader_1x02_P2.54mm_Horizontal -> Connector_PinHeader_2.54mm:PinHeader_1x02_P2.54mm_Vertical
- L2: value 270nH -> 180nH
- Y1: footprint Crystal:Crystal_HC49-4H_Vertical -> Crystal:Crystal_SMD_0603-2Pin_6.0x3.5mm_HandSoldering
Connections:
- net +3V3: now also C7.2, FB2.1, U3.6 (VDD), U4.5 (VDD); no longer C11.1, C19.2, C20.1, U1.20 (VD), U1.21 (VA)
- net COL1: now also U2.6 (GP5); no longer U2.7 (GP6)
- net COL2: now also U2.9 (GP8); no longer U2.10 (GP9)
- net FM_ANT: now also D6.3 (VN)
- net GND: now also C7.1, D5.1 (CH1), D6.1 (CH1), J3.S, U3.7 (GND), U4.4 (GND), U5.2 (GND); no longer C11.2, J1.S
- net ROW1: now also U2.7 (GP6); no longer U2.8 (GP7)
- net ROW2: now also U2.8 (GP7); no longer U2.9 (GP8)
- net OUT_R: now reaches J1.R
- net OUT_R: now also R8.1, U4.7 (VO2)
- net OUT_T: now reaches J1.T
- net OUT_T: now also R9.2, U4.8 (VO1)
- net Audio-: now reaches U1.23 (ROUT/[DOUT])
- net Audio-: now also C6.1, C9.1
- net at C14.1: now also D6.2 (VP)
- net Audio+: now reaches U1.24 (LOUT/[DFS])
- net Audio+: now also C5.1, C8.1
- net headphone_enable: now reaches U2.19 (GP28)
- net headphone_enable: now also U4.3 (~{SD})
- net AM_ANT renamed SW
- net SW: now also U5.1 (RF1); no longer C10.2, L1.2
- net Aud_Enable renamed spk_Enable
- net spk_Enable: now also U3.1 (~{SD})
- new net: C5.2, R1.1
- new net: D5.2 (VP), L3.2
- new net: C10.2, D5.3 (VN)
- new net: R1.2, U3.3 (IN+)
- new net: C9.2, R6.1
- new net: C8.2, R4.1
- new net: J1.S, U4.6 (VO3)
- new net: R4.2, R9.1, U4.1 (IN_1)
- new net: R6.2, R8.2, U4.2 (IN_2)
- new net: R2.2, U3.4 (IN-)
- new net: C6.2, R2.1
- new net AM: C11.1, L1.2, U5.3 (RF2)
- new net Ant_Switch: U2.10 (GP9), U5.4 (CTRL)
- new net Common: C11.2, L3.1, U5.5 (RFC)
- new net RF_PWR: C19.2, C20.1, FB2.2, U1.20 (VD), U1.21 (VA), U5.6 (~{CTRL}/~{VDD})
- new net spk_out+: J3.R, U3.5 (OUT+)
- new net spk_out-: J3.T, U3.8 (OUT-)
Other:
- note added: "Audio Amp PAM8302A (Speaker) LM4910 (Headphones)"
- note removed: "Audio Amp PAM8301"
- moved on the sheet: C1, C10, C14, C19, C2, C20, FB1, L1, L2, U1
