File: PCB/Akash Chowa DX.kicad_pcb (KiCad board)
At the start: 4 copper layers, 110.8 x 70.9 mm, 60 parts, among them J1 Headset, J2 OLED, J3 Speaker, J4 Battery Connection, J5 Conn_01x01_Socket, SW1 EC11 Encoder/SW, SW2 SW_Push, SW3 SW_Push, SW4 SW_Push, SW5 SW_Push, SW6 SW_Push, SW7 SW_Push, U1 Si4735-D60-GU, U2 RP2040-ZERO, U3 PAM8302AAY, U4 LM4910MM, U5 PE4259, Y1 32.768 kHz

Commit message: Adding More parts to the BOM
Parts:
- C12: value 100nF -> 0.1uF
- R1, R2, R3, R4, R5, R6, R8, R9: footprint Resistor_SMD:R_0603_1608Metric_Pad0.98x0.95mm_HandSolder -> Resistor_SMD:R_1206_3216Metric_Pad1.30x1.75mm_HandSolder
- moved R3 1.56 mm to (147.3, 42.8)
- moved R9 1.38 mm to (117.3, 49.5)
- moved C9 0.94 mm to (111.0, 55.1)
- moved C8 0.93 mm to (111.0, 53.3)
- moved C5 0.83 mm to (94.4, 52.0)
- moved C6 0.83 mm to (94.2, 54.1)
- moved R8 0.81 mm to (125.3, 51.5)
- moved R6 0.65 mm to (115.2, 55.7)
- moved R1 0.25 mm to (98.7, 51.7)
Routing:
- net VBUS: track 14.9 -> 17.1 mm
- net Net-(U4-IN_2): track 14.3 -> 12.8 mm
- net /Audio-: track 26.7 -> 27.8 mm
- net /OUT_L: track 9.18 -> 10.0 mm
- net Net-(U3-IN-): track 7.48 -> 6.84 mm
- net Net-(C9-Pad2): track 1.54 -> 2.16 mm
- net batt_read: track 15.6 -> 16.1 mm

Commit message: Finished Adding all parts to Bom
Parts:
- C8, C9: value 0.39uF -> 0.47uF
Changed lines of the file:
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@@
 			)
 		)
-		(property "Value" "0.39uF"
+		(property "Value" "0.47uF"
 			(at 0 1.43 0)
 			(layer "F.Fab")
@@
 			)
 		)
-		(property "Value" "0.39uF"
+		(property "Value" "0.47uF"
 			(at 0 1.43 0)
 			(layer "F.Fab")

Commit message: Adding new stuff after changing PCB size
Parts:
- removed C8, C9: 0.47uF, Capacitor_SMD:C_0603_1608Metric_Pad1.08x0.95mm_HandSolder
- removed D2, D3, D4, D7, D8, D9: 1N4148WT, Diode_SMD:D_SOD-123F
- removed D5, D6: CM1213A-01SO, Package_TO_SOT_SMD:SOT-23
- removed J1: Headset, Connector_Audio:Jack_3.5mm_CUI_SJ1-3523N_Horizontal
- removed R1, R2: 100, Resistor_SMD:R_1206_3216Metric_Pad1.30x1.75mm_HandSolder
- removed R4, R6, R8, R9: 20k, Resistor_SMD:R_1206_3216Metric_Pad1.30x1.75mm_HandSolder
- removed the REF** at (74.6, 38.6)
- removed the REF** at (81.7, 98.9)
- removed the REF** at (153.8, 60.2)
- removed the REF** at (133.5, 54.9)
- removed U3: PAM8302AAY, Package_DFN_QFN:DFN-8-1EP_3x3mm_P0.65mm_EP1.55x2.4mm
- added D10: PRTR5V0U2X, Package_TO_SOT_SMD:SOT-143, F.Cu at (89.8, 51.5)
- added Diode1: 1N4148, 1N4148:DIOAD753W49L380D172B, F.Cu at (119.1, 89.4)
- added Diode2: 1N4148, 1N4148:DIOAD753W49L380D172B, F.Cu at (100.9, 83.7)
- added Diode3: 1N4148, 1N4148:DIOAD753W49L380D172B, F.Cu at (110.9, 93.2)
- added Diode4: 1N4148, 1N4148:DIOAD753W49L380D172B, F.Cu at (107.2, 87.1)
- added Diode5: 1N4148, 1N4148:DIOAD753W49L380D172B, F.Cu at (89.8, 83.0)
- added Diode6: 1N4148, 1N4148:DIOAD753W49L380D172B, F.Cu at (118.1, 83.0)
- added REF**: MountingHole_3.2mm_M3_DIN965, MountingHole:MountingHole_3.2mm_M3_DIN965, F.Cu at (86.6, 76.3)
- added REF**: MountingHole_3.2mm_M3_DIN965, MountingHole:MountingHole_3.2mm_M3_DIN965, F.Cu at (162.0, 65.0)
- added REF**: MountingHole_3.2mm_M3_DIN965, MountingHole:MountingHole_3.2mm_M3_DIN965, F.Cu at (120.0, 71.6)
- added REF**: MountingHole_3.2mm_M3_DIN965, MountingHole:MountingHole_3.2mm_M3_DIN965, F.Cu at (137.7, 51.3)
- C1: value 10uF -> 2.2uF
- C2, C7: value 0.1uF -> 1uF
- C5, C6: value 1uF -> 0.47uF
- U4: value LM4910MM -> TPA6132A2RTE; footprint LM4910MM:SOP65P490X110-8N -> Package_DFN_QFN:WQFN-16-1EP_3x3mm_P0.5mm_EP1.6x1.6mm_ThermalVias
- moved J5 66.1 mm to (107.6, 36.7), turned to 180 degrees
- moved C12 58.8 mm to (107.7, 41.1), turned to -90 degrees
- moved AE1 28.8 mm to (94.2, 36.1), turned to 90 degrees
- moved C6 21.7 mm to (115.7, 50.8)
- moved AE2 21.4 mm to (85.8, 56.9), turned to 180 degrees
- moved C5 21.3 mm to (115.7, 52.6)
- moved C2 20.9 mm to (124.9, 51.4)
- moved C1 20.8 mm to (124.9, 49.6)
- moved J3 16.0 mm to (120.5, 37.8)
- moved C11 14.2 mm to (87.6, 61.5), turned to -90 degrees
- moved J4 10.8 mm to (138.8, 42.0)
- moved L3 10.5 mm to (92.0, 68.1)
- moved C14 9.30 mm to (95.4, 57.6)
- moved FB1 9.30 mm to (94.6, 55.0)
- moved J2 9.07 mm to (145.2, 83.2)
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Connections:
- C1 pad 1: +3V3 -> GND
- C1 pad 2: GND -> Net-(U4-HPVDD)
- C14 pad 1: Net-(D6-VP) -> FM_ANT
- C2 pad 1: GND -> Net-(U4-CPP)
- C2 pad 2: +3V3 -> Net-(U4-CPN)
- C5 pad 1: /Audio+ -> /Audio-
- C5 pad 2: Net-(C5-Pad2) -> Net-(U4-INR+)
- C6 pad 1: /Audio- -> /Audio+
- C6 pad 2: Net-(C6-Pad2) -> Net-(U4-INL+)
- C7 pad 1: GND -> Net-(U4-HPVSS)
- C7 pad 2: +3V3 -> GND
- L3 pad 2: Net-(D5-VP) -> /Net-(D5-VN)
- U2 pad 19: headphone_enable -> Gain0
- U2 pad 20: spk_Enable -> Gain1
- U2 pad 3: unconnected-(U2-GP2-Pad3) -> headphone_enable
- U4 pad 1: Net-(U4-IN_1) -> GND
- U4 pad 2: Net-(U4-IN_2) -> Net-(U4-INL+)
- U4 pad 3: headphone_enable -> Net-(U4-INR+)
- U4 pad 5: +3V3 -> /spk_out-
- U4 pad 6: Net-(U4-VO3) -> Gain0
- U4 pad 7: /OUT_R -> Gain1
- U4 pad 8: /OUT_L -> Net-(U4-HPVSS)
Routing:
- net spk_Enable: track 63.7 -> 0.00 mm, vias 2 -> 0
- net Gain0: track 0.00 -> 45.5 mm
- net Gain1: track 0.00 -> 45.5 mm
- net /ROW1: track 126.9 -> 87.8 mm, vias 1 -> 0
- net Net-(U4-VO3): track 19.5 -> 0.00 mm
- net GND: track 35.2 -> 54.4 mm, vias 94 -> 85
- net +3V3: track 119.1 -> 101.5 mm, vias 3 -> 2
- net headphone_enable: track 42.7 -> 58.9 mm, vias 2 -> 1
- net /Audio-: track 27.8 -> 14.3 mm
- net /OUT_R: track 13.3 -> 0.00 mm
- net Net-(U4-IN_2): track 12.8 -> 0.00 mm
- net /Audio+: track 27.6 -> 14.8 mm, vias 2 -> 0
- net /RF_PWR: track 42.9 -> 30.2 mm
- net /ROW3: track 108.2 -> 96.7 mm, vias 1 -> 0
- net /OUT_L: track 10.0 -> 0.00 mm
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Other:
- board size 110.8 x 70.9 mm -> 98.5 x 70.9 mm
