File: PCB/Akash Chowa DX.kicad_sch (KiCad schematic)
At the start: 56 parts, among them J1 Headset, J2 OLED, J3 Speaker, J4 Battery Connection, J5 Conn_01x01_Socket, SW1 EC11 Encoder/SW, SW2 SW_Push, SW3 SW_Push, SW4 SW_Push, SW5 SW_Push, SW6 SW_Push, SW7 SW_Push, U1 Si4735-D60-GU, U2 RP2040-ZERO, U3 PAM8302AAY, U4 LM4910MM, U5 PE4259, Y1 32.768 kHz

Commit message: Adding More parts to the BOM
Parts:
- C12: value 100nF -> 0.1uF
- C8, C9: value 0.39uF -> 0.47uF
- R1, R2, R3, R4, R5, R6, R8, R9: footprint Resistor_SMD:R_0603_1608Metric_Pad0.98x0.95mm_HandSolder -> Resistor_SMD:R_1206_3216Metric_Pad1.30x1.75mm_HandSolder

Commit message: Adding new stuff after changing PCB size
Parts:
- removed C8, C9: 0.47uF, Capacitor_SMD:C_0603_1608Metric_Pad1.08x0.95mm_HandSolder, symbol Device:C
- removed D2, D3, D4, D7, D8, D9: 1N4148WT, Diode_SMD:D_SOD-123F, symbol Diode:1N4148WT
- removed D5, D6: CM1213A-01SO, Package_TO_SOT_SMD:SOT-23, symbol Power_Protection:CM1213A-01SO
- removed J1: Headset, Connector_Audio:Jack_3.5mm_CUI_SJ1-3523N_Horizontal, symbol Connector_Audio:AudioJack3
- removed R1, R2: 100, Resistor_SMD:R_1206_3216Metric_Pad1.30x1.75mm_HandSolder, symbol Device:R_Small
- removed R4, R6, R8, R9: 20k, Resistor_SMD:R_1206_3216Metric_Pad1.30x1.75mm_HandSolder, symbol Device:R_Small
- removed U3: PAM8302AAY, Package_DFN_QFN:DFN-8-1EP_3x3mm_P0.65mm_EP1.55x2.4mm, symbol Amplifier_Audio:PAM8302AAY
- removed U4: LM4910MM, LM4910MM:SOP65P490X110-8N, symbol LM4910MM:LM4910MM
- added D10: PRTR5V0U2X, Package_TO_SOT_SMD:SOT-143, symbol Power_Protection:PRTR5V0U2X
- added Diode1, Diode2, Diode3, Diode4, Diode5, Diode6: 1N4148, 1N4148:DIOAD753W49L380D172B, symbol 1N4148:1N4148
- added U4: TPA6132A2RTE, Package_DFN_QFN:WQFN-16-1EP_3x3mm_P0.5mm_EP1.6x1.6mm_ThermalVias, symbol Amplifier_Audio:TPA6132A2RTE
- C1: value 10uF -> 2.2uF
- C2, C7: value 0.1uF -> 1uF
- C5, C6: value 1uF -> 0.47uF
Connections:
- net +3V3: now also U4.14 (VDD); no longer C1.1, C2.2, C7.2
- net AM: now also D10.3 (I/O2)
- net Audio+: now also C6.1; no longer C5.1
- net Audio-: now also C5.1; no longer C6.1
- net FM_ANT: now also C14.1
- net GND: now also C1.1, C7.2, D10.1 (GND), D10.4 (VCC), U4.1 (INL-), U4.10 (PGND), U4.15 (SGND), U4.17 (EP), U4.4 (INR-); no longer C1.2, C2.1, C7.1
- net Net-(D5-VN): now also L3.2
- net ROW1: now also Diode1.K, Diode3.K
- net ROW2: now also Diode2.K, Diode4.K
- net ROW3: now also Diode5.K, Diode6.K
- net SW: now also D10.2 (I/O1)
- net headphone_enable: now also U2.3 (GP2), U4.13 (EN); no longer U2.19 (GP28)
- net spk_out+: now also U4.16 (OUTL)
- net spk_out-: now also U4.5 (OUTR)
- net at SW3.2: now also Diode2.A
- net at SW7.2: now also Diode6.A
- net at SW2.2: now also Diode1.A
- net at C5.2: now also U4.3 (INR+)
- net at SW6.2: now also Diode4.A
- net at SW5.2: now also Diode3.A
- net at SW4.2: now also Diode5.A
- net at C6.2: now also U4.2 (INL+)
- net spk_Enable renamed Gain1
- net Gain1: now also U4.7 (G1)
- new net: C1.2, U4.12 (HPVDD)
- new net: C2.1, U4.11 (CPP)
- new net: C7.1, U4.8 (HPVSS)
- new net: C2.2, U4.9 (CPN)
- new net Gain0: U2.19 (GP28), U4.6 (G0)
Other:
- note added: "TPA6132A2RTE AMP for Headphone"
- note removed: "Audio Amp PAM8302A (Speaker) LM4910 (Headphones)"
- moved on the sheet: C6, SW2, SW4, SW5, SW7
